Commit message: add inertial properties to urdf

File: lawnbot_description/urdf/lawnbot.urdf (robot description, URDF)
Before this commit: robot lawnbot, 4 links, 3 joints
Links:
- link base_link: mass None -> 45
- link caster_front: mass None -> 2.2
- link wheel_bl: mass None -> 1.1
- link wheel_br: mass None -> 1.1

Commit message: add launch files, fix build issues, test urdf

File: lawnbot_description/urdf/lawnbot.urdf (robot description, URDF)
Before this commit: robot lawnbot, 4 links, 3 joints
Links:
- link base_link: mass 45 -> None
Joints:
- joint base_to_wheel_bl: origin xyz=0.3 -0.2375 -0.1 rpy=1.5708 3.14159 0 -> xyz=0.3 -0.2375 -0.1 rpy=-1.5708 -3.14159 0
- joint base_to_wheel_br: origin xyz=0.3 0.2375 -0.1 rpy=1.5708 3.14159 0 -> xyz=0.3 0.2375 -0.1 rpy=-1.5708 -3.14159 0

Commit message: add laser to model and gazebo launch files

File: lawnbot_description/urdf/lawnbot.urdf (robot description, URDF)
Before this commit: robot lawnbot, 4 links, 3 joints
Links:
- added link laser_link, mass 1e-5; collision cylinder length=0.05 radius=0.025; visual cylinder length=0.05 radius=0.025
Joints:
- added joint base_to_laser: type fixed, parent base_link, child laser_link, origin xyz=0 0 0.175 rpy=0 0 0
- joint base_to_wheel_bl: origin xyz=0.3 -0.2375 -0.1 rpy=-1.5708 -3.14159 0 -> xyz=0.3 -0.2375 -0.1 rpy=1.57 -3.14159 0
- joint base_to_wheel_br: origin xyz=0.3 0.2375 -0.1 rpy=-1.5708 -3.14159 0 -> xyz=0.3 0.2375 -0.1 rpy=1.57 -3.14159 0
